Commit message: A ton of fiddly changes to namespace the warthog topics and frame_ids
Also, add a VLP-16 sensor to the Warthog model.
At some point I would like to refactor this to make it cleaner.

File: warthog_description/urdf/accessories.urdf.xacro (robot description, xacro)
@@ -9,4 +9,8 @@
     warthog_base/launch/base.launch
   -->
+  <xacro:include filename="$(find velodyne_description)/urdf/VLP-16.urdf.xacro"/>
+  <VLP-16 name="velodyne" topic="velodyne_points" framename="warthog/velodyne" parent="top_chassis_link" hz="10" samples="365" gpu="true">
+    <origin xyz="0 0 0.5" rpy="0 0 0"/>
+  </VLP-16>
   <!-- If enabled, generate a Novatel Smart6 payload. -->
   <xacro:include filename="accessories/novatel_smart6.urdf.xacro" />
